File: ramau80aisoworkbench1/ramau80aisoworkbench1.kicad_sch (KiCad schematic)
At the start: 189 parts, among them J1 Conn_01x04_Socket, SW1 SW_PUSH, U1 ATmega32U4-AU, Y1 16MHz

Commit message: all parts on board! lets make sure the resistors and capacitors are all right and that the ground issue is sorted. then routing
Parts:
- J1: footprint (none) -> Connector_JST:JST_SH_SM04B-SRSS-TB_1x04-1MP_P1.00mm_Horizontal
- SW1: footprint random-keyboard-parts:SKQG-1155865 -> random-keyboard-parts:PushButton_6x6mm_TH_Pretty
Changed lines of the file:
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@@
       (effects (font (size 1.27 1.27)))
     )
-    (property "Footprint" "random-keyboard-parts:SKQG-1155865" (at 119.38 148.59 0)
+    (property "Footprint" "random-keyboard-parts:PushButton_6x6mm_TH_Pretty" (at 119.38 148.59 0)
       (effects (font (size 1.524 1.524)) hide)
     )
@@
       (effects (font (size 1.27 1.27)) (justify left))
     )
-    (property "Footprint" "" (at 148.59 175.26 0)
+    (property "Footprint" "Connector_JST:JST_SH_SM04B-SRSS-TB_1x04-1MP_P1.00mm_Horizontal" (at 148.59 175.26 0)
       (effects (font (size 1.27 1.27)) hide)
     )
