File: ramau80aisoworkbench1/ramau80aisoworkbench1.kicad_pcb (KiCad board)
At the start: 2 copper layers, 357.5 x 128.8 mm, 190 parts, among them J1 Conn_01x04_Socket, SW1 SW_PUSH, U1 ATmega32U4-AU, Y1 16MHz

Commit message: more traces
Routing:
- net +5V: track 163.4 -> 241.2 mm, vias 6 -> 8
- net Net-(U1-~{RESET}): track 0.00 -> 52.2 mm, vias 0 -> 2
Changed lines of the file:
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@@
   (segment (start 30.48 17.145) (end 99.695 17.145) (width 0.25) (layer "F.Cu") (net 1))
   (segment (start 118.25 32) (end 119.25 31) (width 0.25) (layer "F.Cu") (net 1))
+  (segment (start 131.106302 26.67) (end 130.81 26.67) (width 0.25) (layer "F.Cu") (net 1))
+  (segment (start 130.81 26.67) (end 129.54 25.4) (width 0.25) (layer "F.Cu") (net 1))
+  (segment (start 116.765 41.2) (end 116.55 41.2) (width 0.25) (layer "F.Cu") (net 1))
   (via (at 123.25 32) (size 0.8) (drill 0.4) (layers "F.Cu" "B.Cu") (net 1))
   (via (at 129 26.25) (size 0.8) (drill 0.4) (layers "F.Cu" "B.Cu") (net 1))
@@
   (via (at 107.315 13.97) (size 0.8) (drill 0.4) (layers "F.Cu" "B.Cu") (net 1))
   (via (at 118.25 32) (size 0.8) (drill 0.4) (layers "F.Cu" "B.Cu") (net 1))
+  (via (at 131.106302 26.67) (size 0.8) (drill 0.4) (layers "F.Cu" "B.Cu") (net 1))
+  (via (at 129.54 25.4) (size 0.8) (drill 0.4) (layers "F.Cu" "B.Cu") (net 1))
+  (segment (start 122.285 18.2) (end 123.16 18.2) (width 0.25) (layer "B.Cu") (net 1))
+  (segment (start 114.93 12.7) (end 114.26 13.37) (width 0.25) (layer "B.Cu") (net 1))
+  (segment (start 121.285 19.6) (end 122.285 20.6) (width 0.25) (layer "B.Cu") (net 1))
+  (segment (start 121.46 15.7) (end 121.46 17.375) (width 0.25) (layer "B.Cu") (net 1))
+  (segment (start 122.285 22.2) (end 123.16 22.2) (width 0.25) (layer "B.Cu") (net 1))
+  (segment (start 127 29.5) (end 127 29.25) (width 0.25) (layer "B.Cu") (net 1))
   (segment (start 119.86 27.975) (end 119.86 27.1) (width 0.25) (layer "B.Cu") (net 1))
+  (segment (start 134.625 24.125) (end 133.75 23.25) (width 0.25) (layer "B.Cu") (net 1))
+  (segment (start 129.54 25.4) (end 129.54 25.71) (width 0.25) (layer "B.Cu") (net 1))
   (segment (start 22.86 7.62) (end 22.86 9.525) (width 0.25) (layer "B.Cu") (net 1))
   (segment (start 126.66 22.2) (end 123.16 22.2) (width 0.25) (layer "B.Cu") (net 1))
+  (segment (start 122.085 22) (end 122.285 22.2) (width 0.25) (layer "B.Cu") (net 1))
+  (segment (start 123.16 18.2) (end 122.16 18.2) (width 0.25) (layer "B.Cu") (net 1))
   (segment (start 119.75 32) (end 118.25 32) (width 0.25) (layer "B.Cu") (net 1))
+  (segment (start 115.48 29.935) (end 115.66 29.755) (width 0.25) (layer "B.Cu") (net 1))
   (segment (start 120.66 15.7) (end 120.66 13.01) (width 0.25) (layer "B.Cu") (net 1))
+  (segment (start 134 31.25) (end 133.7 30.95) (width 0.25) (layer "B.Cu") (net 1))
+  (segment (start 133.7 30.95) (end 133.7 28.2) (width 0.25) (layer "B.Cu") (net 1))
+  (segment (start 114.26 13.37) (end 114.26 15.7) (width 0.25) (layer "B.Cu") (net 1))
+  (segment (start 132.7 22.2) (end 127.34 22.2) (width 0.25) (layer "B.Cu") (net 1))
   (segment (start 126.75 29) (end 120.885 29) (width 0.25) (layer "B.Cu") (net 1))
+  (segment (start 134.625 27.275) (end 134.625 24.125) (width 0.25) (layer "B.Cu") (net 1))
+  (segment (start 133.7 28.2) (end 134.625 27.275) (width 0.25) (layer "B.Cu") (net 1))
+  (segment (start 121.46 17.375) (end 122.285 18.2) (width 0.25) (layer "B.Cu") (net 1))
   (segment (start 133.95 27.95) (end 134.05 27.95) (width 0.25) (layer "B.Cu") (net 1))
   (segment (start 110.38 24.13) (end 110.85 24.6) (width 0.25) (layer "B.Cu") (net 1))
+  (segment (start 118.25 31.255) (end 118.25 32) (width 0.25) (layer "B.Cu") (net 1))
+  (segment (start 116.75 29.755) (end 118.25 31.255) (width 0.25) (layer "B.Cu") (net 1))
+  (segment (start 122.87 12.7) (end 120.66 14.91) (width 0.25) (layer "B.Cu") (net 1))
+  (segment (start 109.22 15.24) (end 108.585 15.24) (width 0.25) (layer "B.Cu") (net 1))
   (segment (start 112.395 13.97) (end 113.46 15.035) (width 0.25) (layer "B.Cu") (net 1))
+  (segment (start 122.085 20.79) (end 122.085 22) (width 0.25) (layer "B.Cu") (net 1))
+  (segment (start 122.16 18.2) (end 121.285 19.075) (width 0.25) (layer "B.Cu") (net 1))
+  (segment (start 120.66 14.91) (end 120.66 15.7) (width 0.25) (layer "B.Cu") (net 1))
   (segment (start 113.46 15.035) (end 113.46 15.7) (width 0.25) (layer "B.Cu") (net 1))
   (segment (start 127 29.5) (end 129 27.5) (width 0.25) (layer "B.Cu") (net 1))
   (segment (start 120.66 13.01) (end 120.97 12.7) (width 0.25) (layer "B.Cu") (net 1))
   (segment (start 109.22 26.03) (end 109.85 25.4) (width 0.25) (layer "B.Cu") (net 1))
+  (segment (start 108.585 15.24) (end 107.315 13.97) (width 0.25) (layer "B.Cu") (net 1))
   (segment (start 114.26 13.93) (end 114.26 15.7) (width 0.25) (layer "B.Cu") (net 1))
+  (segment (start 122.275 20.6) (end 122.085 20.79) (width 0.25) (layer "B.Cu") (net 1))
   (segment (start 109.22 24.13) (end 110.38 24.13) (width 0.25) (layer "B.Cu") (net 1))
+  (segment (start 129.54 25.71) (end 129 26.25) (width 0.25) (layer "B.Cu") (net 1))
+  (segment (start 111.76 28.575) (end 111.76 25.4) (width 0.25) (layer "B.Cu") (net 1))
+  (segment (start 133.75 23.25) (end 132.7 22.2) (width 0.25) (layer "B.Cu") (net 1))
   (segment (start 120.885 29) (end 119.86 27.975) (width 0.25) (layer "B.Cu") (net 1))
   (segment (start 121.65 32) (end 123.25 32) (width 0.25) (layer "B.Cu") (net 1))
+  (segment (start 116.55 41.2) (end 116.55 39.081396) (width 0.25) (layer "B.Cu") (net 1))
+  (segment (start 127.34 22.2) (end 127 22.54) (width 0.25) (layer "B.Cu") (net 1))
   (segment (start 22.86 9.525) (end 30.48 17.145) (width 0.25) (layer "B.Cu") (net 1))
+  (segment (start 127 29.25) (end 126.75 29) (width 0.25) (layer "B.Cu") (net 1))
   (segment (start 131.65 26.25) (end 131.75 26.25) (width 0.25) (layer "B.Cu") (net 1))
   (segment (start 127 22.54) (end 126.66 22.2) (width 0.25) (layer "B.Cu") (net 1))
+  (segment (start 121.285 19.075) (end 121.285 19.6) (width 0.25) (layer "B.Cu") (net 1))
   (segment (start 113.46 13.13) (end 113.03 12.7) (width 0.25) (layer "B.Cu") (net 1))
+  (segment (start 132 26) (end 131.965 26.035) (width 0.25) (layer "B.Cu") (net 1))
+  (segment (start 115.48 38.011396) (end 115.48 29.935) (width 0.25) (layer "B.Cu") (net 1))
   (segment (start 129 27.5) (end 129 26.25) (width 0.25) (layer "B.Cu") (net 1))
   (segment (start 113.03 12.7) (end 114.26 13.93) (width 0.25) (layer "B.Cu") (net 1))
+  (segment (start 128 26.25) (end 128 23.54) (width 0.25) (layer "B.Cu") (net 1))
+  (segment (start 131.965 26.035) (end 131.741302 26.035) (width 0.25) (layer "B.Cu") (net 1))
+  (segment (start 114.93 12.7) (end 120.97 12.7) (width 0.25) (layer "B.Cu") (net 1))
+  (segment (start 115.66 29.755) (end 112.94 29.755) (width 0.25) (layer "B.Cu") (net 1))
   (segment (start 119.06 28.06) (end 120.5 29.5) (width 0.25) (layer "B.Cu") (net 1))
   (segment (start 128 26.25) (end 128 27.75) (width 0.25) (layer "B.Cu") (net 1))
   (segment (start 119.06 27.1) (end 119.06 28.06) (width 0.25) (layer "B.Cu") (net 1))
   (segment (start 128 27.75) (end 126.75 29) (width 0.25) (layer "B.Cu") (net 1))
+  (segment (start 122.285 20.6) (end 123.16 20.6) (width 0.25) (layer "B.Cu") (net 1))
+  (segment (start 120.66 15.7) (end 121.46 15.7) (width 0.25) (layer "B.Cu") (net 1))
+  (segment (start 128 23.54) (end 127 22.54) (width 0.25) (layer "B.Cu") (net 1))
   (segment (start 109.85 25.4) (end 111.76 25.4) (width 0.25) (layer "B.Cu") (net 1))
+  (segment (start 112.94 29.755) (end 111.76 28.575) (width 0.25) (layer "B.Cu") (net 1))
+  (segment (start 131.741302 26.035) (end 131.106302 26.67) (width 0.25) (layer "B.Cu") (net 1))
+  (segment (start 116.55 39.081396) (end 115.48 38.011396) (width 0.25) (layer "B.Cu") (net 1))
+  (segment (start 123.16 20.6) (end 122.275 20.6) (width 0.25) (layer "B.Cu") (net 1))
+  (segment (start 115.66 29.755) (end 116.75 29.755) (width 0.25) (layer "B.Cu") (net 1))
   (segment (start 107.315 13.97) (end 112.395 13.97) (width 0.25) (layer "B.Cu") (net 1))
   (segment (start 110.85 24.6) (end 111.76 24.6) (width 0.25) (layer "B.Cu") (net 1))
@@
   (segment (start 125.6405 7.5305) (end 125.6405 15.24) (width 0.25) (layer "B.Cu") (net 118))
   (segment (start 41.275 0) (end 116.84 0) (width 0.25) (layer "B.Cu") (net 118))
+  (segment (start 122.7454 30.48) (end 126.1427 27.0827) (width 0.25) (layer "F.Cu") (net 119))
+  (segment (start 116.205 30.48) (end 122.7454 30.48) (width 0.25) (layer "F.Cu") (net 119))
+  (via (at 116.205 30.48) (size 0.8) (drill 0.4) (layers "F.Cu" "B.Cu") (net 119))
+  (via (at 126.1427 27.0827) (size 0.8) (drill 0.4) (layers "F.Cu" "B.Cu") (net 119))
+  (segment (start 126.1427 28.1623) (end 125.755 28.55) (width 0.25) (layer "B.Cu") (net 119))
+  (segment (start 113.275 48.925) (end 117.057412 48.925) (width 0.25) (layer "B.Cu") (net 119))
+  (segment (start 118.825 46.99) (end 120.73 48.895) (width 0.25) (layer "B.Cu") (net 119))
+  (segment (start 118.825 47.157412) (end 118.825 46.99) (width 0.25) (layer "B.Cu") (net 119))
+  (segment (start 125.755 28.55) (end 121.235 28.55) (width 0.25) (layer "B.Cu") (net 119))
+  (segment (start 126.1427 27.0827) (end 126.1427 28.1623) (width 0.25) (layer "B.Cu") (net 119))
+  (segment (start 121.235 28.55) (end 120.66 27.975) (width 0.25) (layer "B.Cu") (net 119))
+  (segment (start 112.05 47.7) (end 113.275 48.925) (width 0.25) (layer "B.Cu") (net 119))
+  (segment (start 117.057412 48.925) (end 118.825 47.157412) (width 0.25) (layer "B.Cu") (net 119))
+  (segment (start 121.285 48.895) (end 122.555 47.625) (width 0.25) (layer "B.Cu") (net 119))
+  (segment (start 122.555 47.625) (end 122.555 44.45) (width 0.25) (layer "B.Cu") (net 119))
+  (segment (start 122.555 44.45) (end 116.205 38.1) (width 0.25) (layer "B.Cu") (net 119))
+  (segment (start 120.73 48.895) (end 121.285 48.895) (width 0.25) (layer "B.Cu") (net 119))
+  (segment (start 120.66 27.975) (end 120.66 27.1) (width 0.25) (layer "B.Cu") (net 119))
+  (segment (start 116.205 38.1) (end 116.205 30.48) (width 0.25) (layer "B.Cu") (net 119))
   (segment (start 111.76 17.4) (end 109.555 17.4) (width 0.25) (layer "B.Cu") (net 120))
   (segment (start 109.555 17.4) (end 109.22 17.065) (width 0.25) (layer "B.Cu") (net 120))
